Commit message: Imported upstream version '0.1.9' of 'upstream'

File: pepper_description/urdf/pepper1.0_generated_urdf/pepper.urdf (robot description, URDF)
Before this commit: robot JulietteY20MP, 84 links, 83 joints
Links:
- removed link ImuBaseGyrometer_frame
Joints:
- removed joint GyrometerBase_sensor_fixedjoint
- joint AccelerometerBase_sensor_fixedjoint: origin xyz=0 0 -0.3 rpy=0 0 0 -> xyz=0.0147 -0.0017 -0.26319 rpy=0 0 0
- joint CameraBottom_sensor_fixedjoint: origin xyz=0.0936 0 0.0616 rpy=0 0.698132 0 -> xyz=0.09262 0 0.06177 rpy=0 0.698132 0
- joint CameraTop_sensor_fixedjoint: origin xyz=0.0868 0 0.1631 rpy=0 0 0 -> xyz=0.08601 0 0.16284 rpy=0 0 0
- joint LaserSensor/Front_sensor_fixedjoint: origin xyz=0.0562 0 -0.0692 rpy=0 0.349044 0 -> xyz=0.0562 0 -0.0692 rpy=0 0.349066 0
- joint LaserSensor/Left_sensor_fixedjoint: origin xyz=-0.018 0.0899 -0.0759 rpy=8.34035e-09 0.191982 1.5708 -> xyz=-0.018 0.0899 -0.0759 rpy=0 0.349066 1.5708
- joint LaserSensor/Right_sensor_fixedjoint: origin xyz=-0.018 -0.0899 -0.0759 rpy=4.08851e-07 0.191857 -1.60746 -> xyz=-0.018 -0.0899 -0.0759 rpy=0 0.349066 -1.5708
- joint LaserSensor/Shovel_sensor_fixedjoint: origin xyz=0.0562 0 -0.0692 rpy=0 0.349044 0 -> xyz=0.0562 0 -0.0692 rpy=0 0.349066 0
- joint LaserSensor/VerticalLeft_sensor_fixedjoint: origin xyz=0.0562 0 -0.0692 rpy=0 0.349044 0 -> xyz=0.0562 0 -0.0692 rpy=0 0.349066 0
- joint LaserSensor/VerticalRight_sensor_fixedjoint: origin xyz=0.0562 0 -0.0692 rpy=0 0.349044 0 -> xyz=0.0562 0 -0.0692 rpy=0 0.349066 0

File: pepper_description/urdf/pepper1.0_generated_urdf/pepper_arms.xacro (robot description, xacro)
@@ -14,5 +14,5 @@
 		<inertial>
 			<mass value="0.3125"/>
-			<inertia ixx="0.000361198" ixy="-1.0453e-07" ixz="-5.24532e-07" iyy="0.000137229" iyz="-5.79522e-06" izz="0.000399194"/>
+			<inertia ixx="0.000361198" ixy="-1.98347e-06" ixz="6.35907e-07" iyy="0.000137229" iyz="-5.68878e-06" izz="0.000399194"/>
 			<origin rpy="0 0 0" xyz="0.00018 -0.01856 0.00099"/>
 		</inertial>
@@ -29,5 +29,5 @@
 		<inertial>
 			<mass value="0.50527"/>
-			<inertia ixx="0.000500872" ixy="0.00109321" ixz="-0.00092282" iyy="0.00126284" iyz="-0.000141027" izz="0.00115718"/>
+			<inertia ixx="0.000500872" ixy="-3.55918e-05" ixz="8.51263e-05" iyy="0.00126284" iyz="9.06813e-06" izz="0.00115718"/>
 			<origin rpy="0 0 0" xyz="0.08151 0.01284 -0.01017"/>
 		</inertial>
@@ -44,5 +44,5 @@
 		<inertial>
 			<mass value="0.27495"/>
-			<inertia ixx="0.000122971" ixy="1.4139e-06" ixz="1.05526e-05" iyy="0.000331766" iyz="1.86491e-06" izz="0.000303047"/>
+			<inertia ixx="0.000122971" ixy="9.86024e-07" ixz="-2.55838e-05" iyy="0.000331766" iyz="-1.98925e-06" izz="0.000303047"/>
 			<origin rpy="0 0 0" xyz="-0.02297 -0.00019 0.00119"/>
 		</inertial>
@@ -59,5 +59,5 @@
 		<inertial>
 			<mass value="0.16579"/>
-			<inertia ixx="0.00156513" ixy="3.85342e-05" ixz="-0.000138805" iyy="0.00173219" iyz="-8.93543e-06" izz="0.000273081"/>
+			<inertia ixx="0.00156513" ixy="1.47517e-05" ixz="-6.05746e-05" iyy="0.00173219" iyz="-1.7619e-07" izz="0.000273081"/>
 			<origin rpy="0 0 0" xyz="0.0593 0.00271 -0.01014"/>
 		</inertial>
@@ -74,5 +74,5 @@
 		<inertial>
 			<mass value="0.27555"/>
-			<inertia ixx="0.000151643" ixy="-2.46935e-05" ixz="-4.3233e-05" iyy="0.000431099" iyz="3.95851e-06" izz="0.000456172"/>
+			<inertia ixx="0.000151643" ixy="1.06629e-05" ixz="2.89509e-06" iyy="0.000431099" iyz="-3.13715e-06" izz="0.000456172"/>
 			<origin rpy="0 0 0" xyz="0.03536 -0.00072 -0.00207"/>
 		</inertial>
@@ -102,5 +102,5 @@
 		<inertial>
 			<mass value="0.3125"/>
-			<inertia ixx="0.000361198" ixy="1.0453e-07" ixz="-5.24532e-07" iyy="0.000137229" iyz="5.79522e-06" izz="0.000399194"/>
+			<inertia ixx="0.000361198" ixy="1.98347e-06" ixz="6.35907e-07" iyy="0.000137229" iyz="5.68878e-06" izz="0.000399194"/>
 			<origin rpy="0 0 0" xyz="0.00018 0.01856 0.00099"/>
 		</inertial>
@@ -117,5 +117,5 @@
 		<inertial>
 			<mass value="0.50527"/>
-			<inertia ixx="0.000500872" ixy="-0.00109321" ixz="-0.00092282" iyy="0.00126284" iyz="0.000141027" izz="0.00115718"/>
+			<inertia ixx="0.000500872" ixy="3.55918e-05" ixz="8.51263e-05" iyy="0.00126284" iyz="-9.06813e-06" izz="0.00115718"/>
 			<origin rpy="0 0 0" xyz="0.08151 -0.01284 -0.01017"/>
 		</inertial>
@@ -132,5 +132,5 @@
 		<inertial>
 			<mass value="0.27495"/>
-			<inertia ixx="0.000122971" ixy="-1.4139e-06" ixz="1.05526e-05" iyy="0.000331766" iyz="-1.86491e-06" izz="0.000303047"/>
+			<inertia ixx="0.000122971" ixy="-9.86024e-07" ixz="-2.55838e-05" iyy="0.000331766" iyz="1.98925e-06" izz="0.000303047"/>
 			<origin rpy="0 0 0" xyz="-0.02297 0.00019 0.00119"/>
 		</inertial>
@@ -147,5 +147,5 @@
 		<inertial>
 			<mass value="0.16579"/>
-			<inertia ixx="0.00156513" ixy="-3.85342e-05" ixz="-0.000138805" iyy="0.00173219" iyz="8.93543e-06" izz="0.000273081"/>
+			<inertia ixx="0.00156513" ixy="-1.47517e-05" ixz="-6.05746e-05" iyy="0.00173219" iyz="1.7619e-07" izz="0.000273081"/>
 			<origin rpy="0 0 0" xyz="0.0593 -0.00271 -0.01014"/>
 		</inertial>
@@ -162,5 +162,5 @@
 		<inertial>
 			<mass value="0.27555"/>
-			<inertia ixx="0.000151643" ixy="2.46935e-05" ixz="-4.3233e-05" iyy="0.000431099" iyz="-3.95851e-06" izz="0.000456172"/>
+			<inertia ixx="0.000151643" ixy="-1.06629e-05" ixz="2.89509e-06" iyy="0.000431099" iyz="3.13715e-06" izz="0.000456172"/>
 			<origin rpy="0 0 0" xyz="0.03536 0.00072 -0.00207"/>
 		</inertial>

File: pepper_description/urdf/pepper1.0_generated_urdf/pepper_fingers.xacro (robot description, xacro)
@@ -32,18 +32,4 @@
 		<mimic joint="LHand" multiplier="0.872665" offset="0"/>
 	</joint>
-	<link name="RFinger11_link">
-		<inertial>
-			<mass value="2e-06"/>
-			<inertia ixx="1.1e-09" ixy="0" ixz="0" iyy="1.1e-09" iyz="0" izz="1.1e-09"/>
-		</inertial>
-		<xacro:insert_visu_RFinger11_link/>
-	</link>
-	<joint name="RFinger11" type="continuous">
-		<parent link="r_wrist"/>
-		<child link="RFinger11_link"/>
-		<origin rpy="1.39757 1.04064 0.0334335" xyz="0.0821 0.0268 0.004"/>
-		<axis xyz="0 0 1.0"/>
-		<mimic joint="RHand" multiplier="0.872665" offset="0"/>
-	</joint>
 	<link name="RFinger12_link">
 		<inertial>
@@ -253,4 +239,18 @@
 		<child link="RFinger23_link"/>
 		<origin rpy="0 0 -1.0472" xyz="0.018 0 0"/>
+		<axis xyz="0 0 1.0"/>
+		<mimic joint="RHand" multiplier="0.872665" offset="0"/>
+	</joint>
+	<link name="RFinger11_link">
+		<inertial>
+			<mass value="2e-06"/>
+			<inertia ixx="1.1e-09" ixy="0" ixz="0" iyy="1.1e-09" iyz="0" izz="1.1e-09"/>
+		</inertial>
+		<xacro:insert_visu_RFinger11_link/>
+	</link>
+	<joint name="RFinger11" type="continuous">
+		<parent link="r_wrist"/>
+		<child link="RFinger11_link"/>
+		<origin rpy="1.39757 1.04064 0.0334335" xyz="0.0821 0.0268 0.004"/>
 		<axis xyz="0 0 1.0"/>
 		<mimic joint="RHand" multiplier="0.872665" offset="0"/>

File: pepper_description/urdf/pepper1.0_generated_urdf/pepper_head.xacro (robot description, xacro)
@@ -14,5 +14,5 @@
 		<inertial>
 			<mass value="0.27391"/>
-			<inertia ixx="0.000343501" ixy="0" ixz="4.87482e-05" iyy="0.000493898" iyz="-2.09863e-06" izz="0.000215252"/>
+			<inertia ixx="0.000343501" ixy="0" ixz="-1.88563e-05" iyy="0.000493898" iyz="2.09863e-06" izz="0.000215252"/>
 			<origin rpy="0 0 0" xyz="-0.00207 0 -0.02636"/>
 		</inertial>
@@ -29,5 +29,5 @@
 		<inertial>
 			<mass value="1.51893"/>
-			<inertia ixx="0.00597209" ixy="0" ixz="0.000931862" iyy="0.0059054" iyz="-4.3428e-07" izz="0.00570374"/>
+			<inertia ixx="0.00597209" ixy="0" ixz="0.000125138" iyy="0.0059054" iyz="4.3428e-07" izz="0.00570374"/>
 			<origin rpy="0 0 0" xyz="0.00312 0 0.11152"/>
 		</inertial>

File: pepper_description/urdf/pepper1.0_generated_urdf/pepper_legs.xacro (robot description, xacro)
@@ -14,5 +14,5 @@
 		<inertial>
 			<mass value="1.02338"/>
-			<inertia ixx="0.00502422" ixy="0" ixz="-1.40621e-05" iyy="0.00640971" iyz="-0.000159449" izz="0.00441082"/>
+			<inertia ixx="0.00502422" ixy="0" ixz="-2.54911e-05" iyy="0.00640971" iyz="0.000159449" izz="0.00441082"/>
 			<origin rpy="0 0 0" xyz="0.00032 0 -0.06039"/>
 		</inertial>
@@ -29,5 +29,5 @@
 		<inertial>
 			<mass value="2.45917"/>
-			<inertia ixx="0.034351" ixy="0" ixz="-0.00134835" iyy="0.0303122" iyz="8.37542e-05" izz="0.0143771"/>
+			<inertia ixx="0.034351" ixy="0" ixz="0.000223034" iyy="0.0303122" iyz="-8.37542e-05" izz="0.0143771"/>
 			<origin rpy="0 0 0" xyz="0.00237 0 -0.09654"/>
 		</inertial>
@@ -44,5 +44,5 @@
 		<inertial>
 			<mass value="11.6015"/>
-			<inertia ixx="0.129229" ixy="0.000401632" ixz="-0.0168449" iyy="0.122839" iyz="-1.01666e-08" izz="0.108168"/>
+			<inertia ixx="0.129229" ixy="-0.000401943" ixz="0.00048556" iyy="0.122839" iyz="-1.01666e-08" izz="0.108168"/>
 			<origin rpy="0 0 0" xyz="0.00220451 0 -0.185729"/>
 		</inertial>

File: pepper_description/urdf/pepper1.0_generated_urdf/pepper_robot.xacro (robot description, xacro)
@@ -12,3 +12,5 @@
 	<xacro:include filename="pepper_fingers.xacro"/>
 	<xacro:include filename="pepper_wheels.xacro"/>
+	<xacro:include filename="pepperGazebo.xacro"/>
+	<xacro:include filename="pepperTransmission.xacro"/>
 </robot>

File: pepper_description/urdf/pepper1.0_generated_urdf/pepper_sensors.xacro (robot description, xacro)
@@ -34,5 +34,5 @@
 		<parent link="Tibia"/>
 		<child link="VerticalLeftLaser_frame"/>
-		<origin rpy="0 0.349044 0" xyz="0.0562 0 -0.0692"/>
+		<origin rpy="0 0.349066 0" xyz="0.0562 0 -0.0692"/>
 		<axis xyz="0 0 0"/>
 	</joint>
@@ -41,5 +41,5 @@
 		<parent link="Tibia"/>
 		<child link="SurroundingFrontLaser_device_frame"/>
-		<origin rpy="0 0.349044 0" xyz="0.0562 0 -0.0692"/>
+		<origin rpy="0 0.349066 0" xyz="0.0562 0 -0.0692"/>
 		<axis xyz="0 0 0"/>
 	</joint>
@@ -62,5 +62,5 @@
 		<parent link="Tibia"/>
 		<child link="ShovelLaser_frame"/>
-		<origin rpy="0 0.349044 0" xyz="0.0562 0 -0.0692"/>
+		<origin rpy="0 0.349066 0" xyz="0.0562 0 -0.0692"/>
 		<axis xyz="0 0 0"/>
 	</joint>
@@ -72,9 +72,9 @@
 		<axis xyz="0 0 0"/>
 	</joint>
-	<link name="CameraTop_frame"/>
-	<joint name="CameraTop_sensor_fixedjoint" type="fixed">
-		<parent link="Head"/>
-		<child link="CameraTop_frame"/>
-		<origin rpy="0 0 0" xyz="0.0868 0 0.1631"/>
+	<link name="RSpeaker_frame"/>
+	<joint name="SpeakerRight_sensor_fixedjoint" type="fixed">
+		<parent link="Head"/>
+		<child link="RSpeaker_frame"/>
+		<origin rpy="0 0 0" xyz="0 0 0"/>
 		<axis xyz="0 0 0"/>
 	</joint>
@@ -83,5 +83,5 @@
 		<parent link="Tibia"/>
 		<child link="SurroundingRightLaser_device_frame"/>
-		<origin rpy="4.08851e-07 0.191857 -1.60746" xyz="-0.018 -0.0899 -0.0759"/>
+		<origin rpy="0 0.349066 -1.5708" xyz="-0.018 -0.0899 -0.0759"/>
 		<axis xyz="0 0 0"/>
 	</joint>
@@ -100,9 +100,9 @@
 		<axis xyz="0 0 0"/>
 	</joint>
-	<link name="ImuBaseGyrometer_frame"/>
-	<joint name="GyrometerBase_sensor_fixedjoint" type="fixed">
-		<parent link="Tibia"/>
-		<child link="ImuBaseGyrometer_frame"/>
-		<origin rpy="0 0 0" xyz="0 0 -0.3"/>
+	<link name="CameraTop_frame"/>
+	<joint name="CameraTop_sensor_fixedjoint" type="fixed">
+		<parent link="Head"/>
+		<child link="CameraTop_frame"/>
+		<origin rpy="0 0 0" xyz="0.08601 0 0.16284"/>
 		<axis xyz="0 0 0"/>
 	</joint>
@@ -111,5 +111,5 @@
 		<parent link="Tibia"/>
 		<child link="SurroundingLeftLaser_device_frame"/>
-		<origin rpy="8.34035e-09 0.191982 1.5708" xyz="-0.018 0.0899 -0.0759"/>
+		<origin rpy="0 0.349066 1.5708" xyz="-0.018 0.0899 -0.0759"/>
 		<axis xyz="0 0 0"/>
 	</joint>
@@ -139,5 +139,5 @@
 		<parent link="Tibia"/>
 		<child link="VerticalRightLaser_frame"/>
-		<origin rpy="0 0.349044 0" xyz="0.0562 0 -0.0692"/>
+		<origin rpy="0 0.349066 0" xyz="0.0562 0 -0.0692"/>
 		<axis xyz="0 0 0"/>
 	</joint>
@@ -160,5 +160,5 @@
 		<parent link="Head"/>
 		<child link="CameraBottom_frame"/>
-		<origin rpy="0 0.698132 0" xyz="0.0936 0 0.0616"/>
+		<origin rpy="0 0.698132 0" xyz="0.09262 0 0.06177"/>
 		<axis xyz="0 0 0"/>
 	</joint>
@@ -173,5 +173,5 @@
 		<parent link="Tibia"/>
 		<child link="ImuBaseAccelerometer_frame"/>
-		<origin rpy="0 0 0" xyz="0 0 -0.3"/>
+		<origin rpy="0 0 0" xyz="0.0147 -0.0017 -0.26319"/>
 		<axis xyz="0 0 0"/>
 	</joint>
@@ -218,11 +218,4 @@
 		<axis xyz="0 0 0"/>
 	</joint>
-	<link name="RSpeaker_frame"/>
-	<joint name="SpeakerRight_sensor_fixedjoint" type="fixed">
-		<parent link="Head"/>
-		<child link="RSpeaker_frame"/>
-		<origin rpy="0 0 0" xyz="0 0 0"/>
-		<axis xyz="0 0 0"/>
-	</joint>
 	<link name="HeadTouchMiddle_frame"/>
 	<joint name="Head/Touch/Middle_sensor_fixedjoint" type="fixed">

File: pepper_description/urdf/pepper1.0_generated_urdf/pepper_torso.xacro (robot description, xacro)
@@ -14,5 +14,5 @@
 		<inertial>
 			<mass value="3.99533"/>
-			<inertia ixx="0.0452761" ixy="0" ixz="-0.00525567" iyy="0.0432702" iyz="0.000266886" izz="0.0258881"/>
+			<inertia ixx="0.0452761" ixy="0" ixz="0.00499091" iyy="0.0432702" iyz="-0.000266886" izz="0.0258881"/>
 			<origin rpy="0 0 0" xyz="0.00322 0 -0.01029"/>
 		</inertial>
